Commit message: True up dimensions and fix rear wheels

File: phoenix_description/urdf/phoenix.urdf (robot description, URDF)
Before this commit: robot phoenix, 11 links, 10 joints
Links:
- removed link rear_wheels
- added link left_rear_wheel; collision cylinder length=0.2032 radius=0.127; visual cylinder length=0.2032 radius=0.127
- added link physical_rear_axle, mass 1; visual cylinder length=0.9398 radius=0.050
- added link right_rear_wheel; collision cylinder length=0.2032 radius=0.127; visual cylinder length=0.2032 radius=0.127
- link base_link: geometry collision box size=1.3967 0.8382 0.1; visual box size=1.3967 0.8382 0.1
- link left_front_wheel: geometry collision cylinder length=0.1143 radius=0.12065; visual cylinder length=0.1143 radius=0.12065
Joints:
- removed joint rear_wheels_to_rear_axle
- added joint left_rear_wheel_to_physical_rear_axle: type fixed, parent physical_rear_axle, child left_rear_wheel, origin xyz=0 0 -0.6371 rpy=0 0 0
- added joint rear_axle_to_physical_rear_axle: type continuous, parent rear_axle, child physical_rear_axle, origin xyz=0 0 0 rpy=1.5708 0 0, axis 0 1 0
- added joint right_rear_wheel_to_physical_rear_axle: type fixed, parent physical_rear_axle, child right_rear_wheel, origin xyz=0 0 0.6371 rpy=0 0 0
- joint base_footprint_to_rear_axle: origin xyz=0 0 0.09525 rpy=0 0 0 -> xyz=0 0 0.127 rpy=0 0 0
- joint left_front_wheel_steer: origin xyz=0.619075 0.6477 -0.054 rpy=0 0 0 -> xyz=1.03505 0.6477 -0.054 rpy=0 0 0; parent base_link -> rear_axle
- joint rear_axle_to_base_link: origin xyz=0.78 0 0.09525 rpy=0 0 0 -> xyz=0.82535 0 0 rpy=0 0 0
- joint right_front_wheel_steer: origin xyz= 0.619075 -0.6477 -0.054 rpy=0 0 0 -> xyz=1.03505 -0.6477 -0.054 rpy=0 0 0; parent base_link -> rear_axle

Commit message: More fixes lol

File: phoenix_description/urdf/phoenix.urdf (robot description, URDF)
Before this commit: robot phoenix, 13 links, 12 joints
Links:
- link left_cam_link: mass 90 -> 0.1
- link mid_cam_link: mass 90 -> 0.1
- link physical_rear_axle: mass 1 -> 10
- link right_cam_link: mass 90 -> 0.1
- link right_front_wheel: geometry collision cylinder length=0.1143 radius=0.12065; visual cylinder length=0.1143 radius=0.12065
Joints:
- joint left_front_wheel_steer: origin xyz=1.03505 0.6477 -0.054 rpy=0 0 0 -> xyz=1.03505 0.6477 0 rpy=0 0 0
- joint rear_axle_to_physical_rear_axle: axis 0 1 0 -> 0 0 1
- joint right_front_wheel_steer: origin xyz=1.03505 -0.6477 -0.054 rpy=0 0 0 -> xyz=1.03505 -0.6477 0 rpy=0 0 0

Commit message: Fixed inertial values

File: phoenix_description/urdf/phoenix.urdf (robot description, URDF)
Before this commit: robot phoenix, 13 links, 12 joints
Links:
- link left_front_wheel: mass 0.1 -> 1.1
- link right_front_wheel: mass 0.1 -> 1.1

Commit message: Adjusted ackermann plugin settings and fixed backwards movement

File: phoenix_description/urdf/phoenix.urdf (robot description, URDF)
Before this commit: robot phoenix, 13 links, 12 joints
Joints:
- joint base_footprint_to_rear_axle: origin xyz=0 0 0.127 rpy=0 0 0 -> xyz=0 0 0.127 rpy=3.14159 0 0

Commit message: more stuff lol

File: phoenix_description/urdf/phoenix.urdf (robot description, URDF)
Before this commit: robot phoenix, 13 links, 12 joints
Joints:
- joint base_footprint_to_rear_axle: origin xyz=0 0 0.127 rpy=3.14159 0 0 -> xyz=0 0 0.127 rpy=0 0 0
- joint rear_axle_to_physical_rear_axle: origin xyz=0 0 0 rpy=1.5708 0 0 -> xyz=0 0 0 rpy=1.5708 0 3.14159

Commit message: Create good area and sky cam It appears that the good areas are not actually aligned even though the image was. Topics also still need to be renamed.

File: phoenix_description/urdf/phoenix.urdf (robot description, URDF)
Before this commit: robot phoenix, 13 links, 12 joints
Links:
- added link sky_cam_link, mass 0.1; visual box size=0.02 0.05 0.02
Joints:
- added joint sky_cam_to_base_link: type fixed, parent base_footprint, child sky_cam_link, origin xyz=0 0 20.5 rpy=0 1.57 0

Commit message: Remove all cameras but mid, and remap topics.

File: phoenix_description/urdf/phoenix.urdf (robot description, URDF)
Before this commit: robot phoenix, 14 links, 13 joints
Links:
- removed link left_cam_link
- removed link right_cam_link
Joints:
- removed joint left_cam_to_rear_axle
- removed joint right_cam_to_rear_axle

Commit message: Changed plugin file paths to match gz namespace change + minor steering adjustments

File: phoenix_description/urdf/phoenix.urdf (robot description, URDF)
Before this commit: robot phoenix, 12 links, 11 joints
Joints:
- joint left_front_wheel_steer: limit lower=-0.3499 upper=+0.5236 effort=0.88269 velocity=3.0 -> lower=-0.3499 upper=+0.5236 effort=25 velocity=3.141
- joint right_front_wheel_steer: limit lower=-0.3499 upper=+0.5236 effort=0.88269 velocity=3.0 -> lower=-0.3499 upper=+0.5236 effort=25 velocity=3.141

Commit message: Attempt to get webots working

File: phoenix_description/urdf/phoenix.urdf (robot description, URDF)
Before this commit: robot phoenix, 12 links, 11 joints
Links:
- removed link sky_cam_link
- link left_front_wheel_rack: geometry visual box size=0.001 0.001 0.001
- link rear_axle: geometry visual box size=0.001 0.001 0.001
- link right_front_wheel_rack: geometry visual box size=0.001 0.001 0.001
Joints:
- removed joint sky_cam_to_base_link

Commit message: Add lidar

File: phoenix_description/urdf/phoenix.urdf (robot description, URDF)
Before this commit: robot phoenix, 11 links, 10 joints
Links:
- added link lidar_link, mass 2.2; collision cylinder length=0.1636 radius=0.0498; visual cylinder length=0.1636 radius=0.0498
Joints:
- added joint lidar_to_rear_axel: type fixed, parent rear_axle, child lidar_link, origin xyz=1.4 0 0.25 rpy=0 0 0

Commit message: Move to using two cameras

File: phoenix_description/urdf/phoenix.urdf (robot description, URDF)
Before this commit: robot phoenix, 12 links, 11 joints
Links:
- added link left_cam_link, mass 0.1; collision box size=0.02 0.05 0.02; visual box size=0.02 0.05 0.02
- added link right_cam_link, mass 0.1; collision box size=0.02 0.05 0.02; visual box size=0.02 0.05 0.02
Joints:
- added joint left_cam_to_mid_cam: type fixed, parent mid_cam_link, child left_cam_link, origin xyz=0 0.2 0 rpy=0 0 0.785398
- added joint right_cam_to_mid_cam: type fixed, parent mid_cam_link, child right_cam_link, origin xyz=0 -0.2 0 rpy=0 0 -0.785398

Commit message: Find better location

File: phoenix_description/urdf/phoenix.urdf (robot description, URDF)
Before this commit: robot phoenix, 14 links, 13 joints
Joints:
- joint left_cam_to_mid_cam: origin xyz=0 0.2 0 rpy=0 0 0.785398 -> xyz=0 0.2 0 rpy=0 0 0.585398
- joint right_cam_to_mid_cam: origin xyz=0 -0.2 0 rpy=0 0 -0.785398 -> xyz=0 -0.2 0 rpy=0 0 -0.585398

Commit message: updating SIM for GPS

File: phoenix_description/urdf/phoenix.urdf (robot description, URDF)
Before this commit: robot phoenix, 14 links, 13 joints
Links:
- added link vectornav; visual box size=0.05 0.05 0.05
Joints:
- added joint vectornav_to_rear_axle: type fixed, parent rear_axle, child vectornav, origin xyz=1.0 0 0.5 rpy=0 0 0

Commit message: Alex's wonderful changes of many lines
- remapped gps topics to match
- added in imu frame for tf2 tree
- over wrote imu0 to use defualt covarance matrix
	- this is because navsat needs non zero covarance
	- idk why just put the gps cord in the frame lit bro

File: phoenix_description/urdf/phoenix.urdf (robot description, URDF)
Before this commit: robot phoenix, 15 links, 14 joints
Links:
- added link imu_link, mass 0.001; visual box size=0.001 0.001 0.001
Joints:
- added joint imu_link_to_vectornav: type fixed, parent vectornav, child imu_link, origin xyz=0 0 0 rpy=0 0 0
